File: schematic/keg01/keg01.sch (KiCad schematic (older format))
At the start: 39 parts, among them IC1 ESP-12E, IC2 HX711_SHL, IC3 AP2112K-3.3, P1 Conn_01x03, P2 Conn_01x03, P3 Conn_01x03, P4 Conn_01x03, P5 Conn_01x02, P6 Conn_01x04, X1 NA

Commit message: layout
Connections:
- net +3V3: no longer R1.1, R5.1
- net PWIC1: now reaches C3.1, C4.1, FB1.1, IC1.8 (VCC)
- net PWIC1: now also R1.1
- net PWIC2: now reaches C12.1, C13.1, FB2.1, IC2.5 (VCC)
- net PWIN2: now reaches C5.1, C6.1, C7.1, D1.1 (K), IC3.1 (VIN), R3.2
- net PWIN: now reaches D1.2 (A), P5.2 (Pin_2)
- net PWDISP: now reaches C16.1, C17.1, FB3.1, P6.2 (Pin_2)
- net PWDISP: now also R5.1
Changed lines of the file:
@@
 U 1 1 5FF2E49F
 P 3000 5300
-F 0 "R1" H 3059 5346 50  0000 L CNN
-F 1 "10k" H 3059 5255 50  0000 L CNN
+F 0 "R1" H 2850 5350 50  0000 L CNN
+F 1 "10k" H 2800 5250 50  0000 L CNN
 F 2 "Resistors_SMD:R_0603" H 3000 5300 50  0001 C CNN
 F 3 "~" H 3000 5300 50  0001 C CNN
@@
 Wire Wire Line
 	3300 5500 3300 5400
-Wire Wire Line
-	3400 5700 3000 5700
-Wire Wire Line
-	3000 5700 3000 5400
 $Comp
 L Device:R_Small R6
@@
 	1    0    0    -1
 $EndComp
-$Comp
-L power:+3V3 #PWR0105
-U 1 1 5FF322D4
-P 3000 5100
-F 0 "#PWR0105" H 3000 4950 50  0001 C CNN
-F 1 "+3V3" H 3015 5273 50  0000 C CNN
-F 2 "" H 3000 5100 50  0001 C CNN
-F 3 "" H 3000 5100 50  0001 C CNN
-	1    3000 5100
-	1    0    0    -1
-$EndComp
 Wire Wire Line
 	5600 5200 5600 5100
 Wire Wire Line
 	3300 5200 3300 5100
-Wire Wire Line
-	3000 5200 3000 5100
 $Comp
 L Connector_Generic:Conn_01x06 X1
@@
 Wire Wire Line
 	5300 6000 5300 5400
-Wire Wire Line
-	5300 5200 5300 5100
-$Comp
-L power:+3V3 #PWR0109
-U 1 1 5FF7A9A2
-P 5300 5100
-F 0 "#PWR0109" H 5300 4950 50  0001 C CNN
-F 1 "+3V3" H 5315 5273 50  0000 C CNN
-F 2 "" H 5300 5100 50  0001 C CNN
-F 3 "" H 5300 5100 50  0001 C CNN
-	1    5300 5100
-	1    0    0    -1
-$EndComp
 $Comp
 L Device:C_Small C13
@@
 Wire Wire Line
 	4300 1500 4700 1500
+Text Label 1800 1500 0    50   ~ 0
+PWIN
+Text Label 2550 1500 0    50   ~ 0
+PWIN2
+Text Label 7500 1500 0    50   ~ 0
+PWIC2
+Text Label 9350 4900 0    50   ~ 0
+PWDISP
+Text Label 2450 6200 0    50   ~ 0
+PWIC1
+Wire Wire Line
+	5300 4800 5300 5200
+Text Label 5300 5100 1    50   ~ 0
+PWDISP
+Wire Wire Line
+	3000 5400 3000 5700
+Wire Wire Line
+	3000 5700 3400 5700
+Wire Wire Line
+	3000 5200 3000 4800
+Text Label 3000 5100 1    50   ~ 0
+PWIC1
 $EndSCHEMATC
