File: schematic/keg02/keg02.sch (KiCad schematic (older format))
At the start: 40 parts, among them IC1 ESP-12E, IC3 AP2112K-3.3, P1 Conn_01x04, P2 Conn_01x03, P5 Conn_01x02, P6 Conn_01x04, X1 NA

Commit message: keg02 rendered image (doc)
Parts:
- IC3: symbol Regulator_Linear:AP2112K-3.3 -> keg02-rescue:AP2112K-3.3-Regulator_Linear
Changed lines of the file:
@@
 	8100 1800 8100 1900
 $Comp
-L Regulator_Linear:AP2112K-3.3 IC3
+L keg02-rescue:AP2112K-3.3-Regulator_Linear IC3
 U 1 1 5FFBFBAB
 P 4400 1600

Commit message: bom update
Parts:
- IC1: symbol ESP8266:ESP-12E -> keg02-rescue:ESP-12E-ESP8266
Changed lines of the file:
@@
 $EndDescr
 $Comp
-L ESP8266:ESP-12E IC1
+L keg02-rescue:ESP-12E-ESP8266 IC1
 U 1 1 5FF2C7EC
 P 4300 5800
